Commit message: Fix build issues, add flexiv_description submodule, add BUILD.md
- Fix CameraInfoManager constructor: pass 'this' instead of get_node_base_interface().get()
- Rewrite cynlr_rizon7_macro to use rizon_arm macro from flexiv_description (Rizon4)
- Update cynlr_arm_system.urdf.xacro to use origin_xyz/rpy string params
- Fix cynlr_system.launch.py: use FindExecutable directly in Command (not PathJoinSubstitution)
- Add flexiv_description as git submodule (humble branch)
- Add BUILD.md with build instructions and next-step guide (URDF xacro parse fix)
- Allow .claude/ settings files in repo

File: cynlr_arm_description/urdf/cynlr_arm_system.urdf.xacro (robot description, xacro)
@@ -26,7 +26,8 @@
     serial_number="$(arg sn_left)"
     vendor="$(arg vendor)"
-    parent="world">
-    <origin xyz="-0.5 0.0 0.9" rpy="0 0 0"/>
-  </xacro:cynlr_rizon7>
+    parent="world"
+    origin_xyz="-0.5 0.0 0.9"
+    origin_rpy="0 0 0"
+  />
   <!-- ------------------------------------------------------------------ -->
   <!-- Center arm — mounted directly above, facing forward                 -->
@@ -36,10 +37,10 @@
     serial_number="$(arg sn_center)"
     vendor="$(arg vendor)"
-    parent="world">
-    <origin xyz="0.0 0.0 1.2" rpy="0 0 0"/>
-  </xacro:cynlr_rizon7>
+    parent="world"
+    origin_xyz="0.0 0.0 1.2"
+    origin_rpy="0 0 0"
+  />
   <!-- ------------------------------------------------------------------ -->
-  <!-- Right arm — mounted at +0.5m on the X axis, rotated 180° to face   -->
-  <!-- the same workspace as the left arm                                  -->
+  <!-- Right arm — mounted at +0.5m on the X axis, rotated 180°           -->
   <!-- ------------------------------------------------------------------ -->
   <xacro:cynlr_rizon7
@@ -47,6 +48,7 @@
     serial_number="$(arg sn_right)"
     vendor="$(arg vendor)"
-    parent="world">
-    <origin xyz="0.5 0.0 0.9" rpy="0 0 3.14159265"/>
-  </xacro:cynlr_rizon7>
+    parent="world"
+    origin_xyz="0.5 0.0 0.9"
+    origin_rpy="0 0 3.14159265"
+  />
 </robot>

File: cynlr_arm_description/urdf/cynlr_rizon7_macro.urdf.xacro (robot description, xacro)
@@ -2,30 +2,42 @@
 <!--
   cynlr_rizon7_macro.urdf.xacro
-  Macro for a single CynLR Rizon-7 arm with ros2_control block.
+  Macro for a single CynLR Rizon 7-DOF arm (Rizon4 variant) with ros2_control block.
   Parameters:
     prefix        – joint/link name prefix, e.g. "arm_left_"
     serial_number – Flexiv serial number (or empty string for sim)
     vendor        – "flexiv" or "sim"
-    parent        – name of the parent link to attach the arm base to
-    *origin       – <origin xyz="..." rpy="..."/> block for base placement
-  Requires flexiv_description to be present in the workspace.
-  Clone: https://github.com/flexivrobotics/flexiv_description  (branch: humble)
+    parent        – parent link to attach the arm base to
+    origin_xyz    – base translation, e.g. "0 0 0"
+    origin_rpy    – base rotation, e.g. "0 0 0"
 -->
 <robot xmlns:xacro="http://www.ros.org/wiki/xacro">
+  <!-- Rizon4 = 7-DOF standard payload arm -->
+  <xacro:property name="rizon_type" value="Rizon4"/>
+  <xacro:include filename="$(find flexiv_description)/urdf/common/rizon_arm.xacro"/>
   <xacro:macro name="cynlr_rizon7"
-               params="prefix serial_number vendor parent *origin">
+               params="prefix serial_number vendor parent
+                       origin_xyz:='0 0 0' origin_rpy:='0 0 0'">
     <!-- ------------------------------------------------------------------ -->
-    <!-- Arm kinematics — provided by flexiv_description                     -->
+    <!-- Arm kinematics — Rizon4 (7-DOF)                                     -->
     <!-- ------------------------------------------------------------------ -->
-    <xacro:include filename="$(find flexiv_description)/urdf/rizon7_macro.urdf.xacro"/>
-    <xacro:rizon7 prefix="${prefix}" parent="${parent}">
-      <xacro:insert_block name="origin"/>
-    </xacro:rizon7>
+    <xacro:rizon_arm
+      prefix="${prefix}"
+      joint_limits_parameters_file="$(find flexiv_description)/config/${rizon_type}/joint_limits.yaml"
+      kinematics_parameters_file="$(find flexiv_description)/config/${rizon_type}/default_kinematics.yaml"
+      inertia_parameters_file="$(find flexiv_description)/config/${rizon_type}/inertia_parameters.yaml"
+      visual_parameters_file="$(find flexiv_description)/config/${rizon_type}/visual_parameters.yaml"
+      add_world_link="false"
+      create_base_joint="false"
+      base_xyz="${origin_xyz}"
+      base_rpy="${origin_rpy}"
+    />
+    <!-- Base joint: attach arm to parent -->
+    <joint name="${prefix}base_joint" type="fixed">
+      <parent link="${parent}"/>
+      <child  link="${prefix}base_link"/>
+      <origin xyz="${origin_xyz}" rpy="${origin_rpy}"/>
+    </joint>
     <!-- ------------------------------------------------------------------ -->
     <!-- ros2_control block — one hardware plugin instance per arm           -->
-    <!--                                                                     -->
-    <!-- All 7 joints expose position + velocity + effort command and state  -->
-    <!-- interfaces. Additional sensor/gpio blocks expose FT, TCP, cartesian,-->
-    <!-- and GPIO interfaces (handled inside CynlrHardwareInterface).        -->
     <!-- ------------------------------------------------------------------ -->
     <ros2_control name="${prefix}system" type="system">
@@ -35,15 +47,13 @@
         <param name="vendor">${vendor}</param>
         <param name="serial_number">${serial_number}</param>
-        <!-- ip_address is optional; leave empty for auto-discovery -->
-        <param name="ip_address"></param>
       </hardware>
-      <!-- 7-DOF arm joints -->
+      <!-- 7 joints: position, velocity, effort -->
       <joint name="${prefix}joint1">
         <command_interface name="position"/>
         <command_interface name="velocity"/>
         <command_interface name="effort"/>
-        <state_interface name="position"/>
-        <state_interface name="velocity"/>
-        <state_interface name="effort"/>
+        <state_interface   name="position"/>
+        <state_interface   name="velocity"/>
+        <state_interface   name="effort"/>
       </joint>
       <joint name="${prefix}joint2">
@@ -51,7 +61,7 @@
         <command_interface name="velocity"/>
         <command_interface name="effort"/>
-        <state_interface name="position"/>
-        <state_interface name="velocity"/>
-        <state_interface name="effort"/>
+        <state_interface   name="position"/>
+        <state_interface   name="velocity"/>
+        <state_interface   name="effort"/>
       </joint>
       <joint name="${prefix}joint3">
@@ -59,7 +69,7 @@
         <command_interface name="velocity"/>
         <command_interface name="effort"/>
-        <state_interface name="position"/>
-        <state_interface name="velocity"/>
-        <state_interface name="effort"/>
+        <state_interface   name="position"/>
+        <state_interface   name="velocity"/>
+        <state_interface   name="effort"/>
       </joint>
       <joint name="${prefix}joint4">
@@ -67,7 +77,7 @@
         <command_interface name="velocity"/>
         <command_interface name="effort"/>
-        <state_interface name="position"/>
-        <state_interface name="velocity"/>
-        <state_interface name="effort"/>
+        <state_interface   name="position"/>
+        <state_interface   name="velocity"/>
+        <state_interface   name="effort"/>
       </joint>
       <joint name="${prefix}joint5">
@@ -75,7 +85,7 @@
         <command_interface name="velocity"/>
         <command_interface name="effort"/>
-        <state_interface name="position"/>
-        <state_interface name="velocity"/>
-        <state_interface name="effort"/>
+        <state_interface   name="position"/>
+        <state_interface   name="velocity"/>
+        <state_interface   name="effort"/>
       </joint>
       <joint name="${prefix}joint6">
@@ -83,7 +93,7 @@
         <command_interface name="velocity"/>
         <command_interface name="effort"/>
-        <state_interface name="position"/>
-        <state_interface name="velocity"/>
-        <state_interface name="effort"/>
+        <state_interface   name="position"/>
+        <state_interface   name="velocity"/>
+        <state_interface   name="effort"/>
       </joint>
       <joint name="${prefix}joint7">
@@ -91,9 +101,9 @@
         <command_interface name="velocity"/>
         <command_interface name="effort"/>
-        <state_interface name="position"/>
-        <state_interface name="velocity"/>
-        <state_interface name="effort"/>
+        <state_interface   name="position"/>
+        <state_interface   name="velocity"/>
+        <state_interface   name="effort"/>
       </joint>
-      <!-- FT sensor state interfaces (raw + ext_tcp + ext_world, 6 channels each) -->
+      <!-- FT sensor state interfaces (18 doubles: raw, ext_tcp, ext_world) -->
       <sensor name="${prefix}ft_sensor">
         <state_interface name="raw_0"/>
@@ -116,5 +126,5 @@
         <state_interface name="ext_world_5"/>
       </sensor>
-      <!-- TCP pose (7) and velocity (6) state interfaces -->
+      <!-- TCP state interfaces (7 pose + 6 velocity = 13 doubles) -->
       <sensor name="${prefix}tcp">
         <state_interface name="pose_0"/>
@@ -132,13 +142,13 @@
         <state_interface name="vel_5"/>
       </sensor>
-      <!-- Full ArmState pointer (for CynlrStateBroadcaster bit_cast trick) -->
+      <!-- Full ArmState pointer — for CynlrStateBroadcaster -->
       <sensor name="${prefix}cynlr_arm_state">
         <state_interface name="full_state_ptr"/>
       </sensor>
-      <!-- Raw ArmInterface pointer (for CynlrNrtPassthroughController) -->
+      <!-- ArmInterface raw pointer — for CynlrNrtPassthroughController (hatch #2) -->
       <sensor name="${prefix}cynlr_arm_ctrl">
         <state_interface name="arm_interface_ptr"/>
       </sensor>
-      <!-- Cartesian command interface (escape hatch #3) -->
+      <!-- Cartesian command interfaces (13 doubles via gpio) — for hatch #3 -->
       <gpio name="${prefix}cartesian_cmd">
         <command_interface name="pose_0"/>
@@ -156,45 +166,4 @@
         <command_interface name="wrench_5"/>
       </gpio>
-      <!-- 18-port digital GPIO -->
-      <gpio name="${prefix}gpio">
-        <!-- Outputs (command) -->
-        <command_interface name="out_0"/>
-        <command_interface name="out_1"/>
-        <command_interface name="out_2"/>
-        <command_interface name="out_3"/>
-        <command_interface name="out_4"/>
-        <command_interface name="out_5"/>
-        <command_interface name="out_6"/>
-        <command_interface name="out_7"/>
-        <command_interface name="out_8"/>
-        <command_interface name="out_9"/>
-        <command_interface name="out_10"/>
-        <command_interface name="out_11"/>
-        <command_interface name="out_12"/>
-        <command_interface name="out_13"/>
-        <command_interface name="out_14"/>
-        <command_interface name="out_15"/>
-        <command_interface name="out_16"/>
-        <command_interface name="out_17"/>
-        <!-- Inputs (state) -->
-        <state_interface name="in_0"/>
-        <state_interface name="in_1"/>
-        <state_interface name="in_2"/>
-        <state_interface name="in_3"/>
-        <state_interface name="in_4"/>
-        <state_interface name="in_5"/>
-        <state_interface name="in_6"/>
-        <state_interface name="in_7"/>
-        <state_interface name="in_8"/>
-        <state_interface name="in_9"/>
-        <state_interface name="in_10"/>
-        <state_interface name="in_11"/>
-        <state_interface name="in_12"/>
-        <state_interface name="in_13"/>
-        <state_interface name="in_14"/>
-        <state_interface name="in_15"/>
-        <state_interface name="in_16"/>
-        <state_interface name="in_17"/>
-      </gpio>
     </ros2_control>
   </xacro:macro>
